File: LMP91000SDX Testing/LMP.kicad_sch (KiCad schematic)
At the start: 1 part, among them U1 LMP91000SDX/NOPB

Commit message: Testing Board Completed
Parts:
- added J1, J2: PPTC071LFBN-RC, PPTC071LFBN_RC:CONN_xPxC071LFBN-RC_SUL, symbol PPTC071LFBN-RC:PPTC071LFBN-RC
- U1: footprint SDA14B -> LMP91000SDX_NOPB:SDA14B
Connections:
- net at U1.1 (DGND): now also J1.7
- net at U1.10 (C1): now also J2.5
- net at U1.11 (VREF): now also J2.4
- net at U1.12 (WE): now also J2.3
- net at U1.13 (RE): now also J2.2
- net at U1.14 (CE): now also J2.1
- net at U1.2 (MENB): now also J1.6
- net at U1.3 (SCL): now also J1.5
- net at U1.4 (SDA): now also J1.4
- net at U1.6 (VDD): now also J1.2
- net at U1.7 (AGND): now also J1.1
- net at U1.8 (VOUT): now also J2.7
- net at U1.9 (C2): now also J2.6
