File: Potensiostat/Battery + Regulator-LAPTOP-311H0TT8.kicad_sch (KiCad schematic)
At the start: 13 parts, among them J2 Conn_01x02_Pin, Q2 Q_PMOS, U3 TP4057, U4 TCR3DF335_LMCT

Commit message: LMP USB Update
Other:
- moved on the sheet: D1, R6
