File: Potensiostat/LMP91000SDX-LAPTOP-311H0TT8.kicad_sch (KiCad schematic)
At the start: 6 parts, among them J1 Conn_01x03_Pin, J3 Conn_01x04_Pin, U2 LMP91000SDX/NOPB

Commit message: LMP USB Update
Parts:
- removed J3: Conn_01x04_Pin, symbol Connector:Conn_01x04_Pin
- R4, R5: value 10k -> R
Other:
- note removed: "Test Pins"
Changed lines of the file:
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@@
 	(rectangle
 		(start 53.34 107.95)
-		(end 81.28 132.334)
-		(stroke
-			(width 0)
-			(type default)
-		)
-		(fill
-			(type none)
-		)
-	)
-	(rectangle
-		(start 83.82 107.95)
-		(end 111.76 132.334)
+		(end 78.232 132.334)
 		(stroke
 			(width 0)
@@
 		(exclude_from_sim no)
 		(at 25.654 21.082 0)
-		(effects
-			(font
-				(size 1.27 1.27)
-			)
-		)
-	)
-	(text "Test Pins"
-		(exclude_from_sim no)
-		(at 91.694 112.014 0)
 		(effects
 			(font
@@
 		)
 	)
-	(label "C2"
-		(at 99.06 127 0)
-		(effects
-			(font
-				(size 1.27 1.27)
-			)
-			(justify left bottom)
-		)
-	)
 	(label "SDA"
 		(at 44.45 76.2 180)
@@
 		)
 	)
-	(label "C1"
-		(at 99.06 124.46 0)
-		(effects
-			(font
-				(size 1.27 1.27)
-			)
-			(justify left bottom)
-		)
-	)
 	(label "SCL"
 		(at 44.45 73.66 180)
@@
 		)
 	)
-	(label "DAC1"
-		(at 99.06 121.92 0)
-		(effects
-			(font
-				(size 1.27 1.27)
-			)
-			(justify left bottom)
-		)
-	)
 	(label "C1"
 		(at 105.41 81.28 0)
@@
 	(label "WE"
 		(at 105.41 76.2 0)
-		(effects
-			(font
-				(size 1.27 1.27)
-			)
-			(justify left bottom)
-		)
-	)
-	(label "ADC1_CH7"
-		(at 99.06 129.54 0)
 		(effects
 			(font
@@
 			)
 		)
-		(property "Value" "10k"
+		(property "Value" "R"
 			(at 43.18 132.0799 0)
 			(effects
@@
 	)
 	(symbol
-		(lib_id "Connector:Conn_01x04_Pin")
-		(at 93.98 124.46 0)
-		(unit 1)
-		(exclude_from_sim no)
-		(in_bom yes)
-		(on_board yes)
-		(dnp no)
-		(fields_autoplaced yes)
-		(property "Reference" "J3"
-			(at 94.615 116.84 0)
-			(effects
-				(font
-					(size 1.27 1.27)
-				)
-			)
-		)
-		(property "Value" "Conn_01x04_Pin"
-			(at 94.615 119.38 0)
-			(effects
-				(font
-					(size 1.27 1.27)
-				)
-			)
-		)
-		(property "Footprint" ""
-			(at 93.98 124.46 0)
-			(effects
-				(font
-					(size 1.27 1.27)
-				)
-				(hide yes)
-			)
-		)
-		(property "Datasheet" "~"
-			(at 93.98 124.46 0)
-			(effects
-				(font
-					(size 1.27 1.27)
-				)
-				(hide yes)
-			)
-		)
-		(property "Description" "Generic connector, single row, 01x04, script generated"
-			(at 93.98 124.46 0)
-			(effects
-				(font
-					(size 1.27 1.27)
-				)
-				(hide yes)
-			)
-		)
-		(pin "4"
-		)
-		(pin "1"
-		)
-		(pin "2"
-		)
-		(pin "3"
-		)
-		(instances
-			(project ""
-				(path "/be108998-ac86-4f7d-931a-841db1905f2a/62dba8b7-8e77-43af-b2ef-391554dc76c9"
-					(reference "J3")
-					(unit 1)
-				)
-			)
-		)
-	)
-	(symbol
 		(lib_id "power:GND")
 		(at 33.02 91.44 0)
@@
 			)
 		)
-		(property "Value" "10k"
+		(property "Value" "R"
 			(at 31.75 132.0799 0)
 			(effects
