File: Helpstat/HELPStat_V2.kicad_sch (KiCad schematic)
At the start: 65 parts, among them IC1 MCP73831/OT, Q1 2.5A/30V/105mΩ

Commit message: Andrew Edits
Parts:
- removed AD5941: AD5941BCPZ-RL7, HELPStat_V2:QFN50P700X700X80-49N, symbol HELPStat_V2-eagle-import:AD5941BCPZ-RL7
- removed BOOT0, RST0: SPST-PTS830GG140, HELPStat_V2:BUTTON-GULLWING, symbol HELPStat_V2-eagle-import:SPST-PTS830GG140
- removed C1, C2: 10u, HELPStat_V2:C0402, symbol HELPStat_V2-eagle-import:CAPACITOR0402
- removed C13, C14, C15, C16: 100n, HELPStat_V2:C0402, symbol HELPStat_V2-eagle-import:CAPACITOR0402
- removed CHRG0: YLW, HELPStat_V2:LED-0603, symbol HELPStat_V2-eagle-import:LED0603
- removed D1: BAT20JFILM, HELPStat_V2:SOD-323, symbol HELPStat_V2-eagle-import:BAT20JFILM
- removed ESP32: ESP32-S3-WROOM-1-N8R8, HELPStat_V2:XCVR_ESP32S3WROOM1N8R8, symbol HELPStat_V2-eagle-import:ESP32-S3-WROOM-1-N8R8
- removed IC1: MCP73831/OT, HELPStat_V2:SOT23-5L, symbol HELPStat_V2-eagle-import:MCP73831/OT
- removed LDO0: AP2112K-3.3TRG1, HELPStat_V2:SOT95P285X140-5N, symbol HELPStat_V2-eagle-import:AP2112K-3.3TRG1
- removed R1: 10k, HELPStat_V2:R0402, symbol HELPStat_V2-eagle-import:RESISTOR0402
- removed R10, R11, R12, R13, R6: 47k, HELPStat_V2:R0402, symbol HELPStat_V2-eagle-import:RESISTOR0402
- removed R2, R3, R5: 4k7, HELPStat_V2:R0402, symbol HELPStat_V2-eagle-import:RESISTOR0402
- removed SDCARD0: MICROSD, HELPStat_V2:MICROSD, symbol HELPStat_V2-eagle-import:MICROSD
- removed TP1, TP2: TEST-POINT3X5, HELPStat_V2:PAD.03X.05, symbol HELPStat_V2-eagle-import:TEST-POINT3X5
- removed USB0: 10118192-0001LF, HELPStat_V2:AMPHENOL_10118192-0001LF, symbol HELPStat_V2-eagle-import:10118192-0001LF
- added C20, C21, C22: 100n, Capacitor_SMD:C_0402_1005Metric, symbol HELPStat_V2-eagle-import:CAPACITOR0402
- added CHRG1: YLW, HELPStat_V2:LED-0603, symbol HELPStat_V2-eagle-import:LED0603
- added D1: BAT20JFILM, BAT20JFILM:SOD-323, symbol BAT20JFILM:BAT20JFILM
- added J1: 10118192-0001LF, 10118192_0001LF:AMPHENOL_10118192-0001LF, symbol 10118192-0001LF:10118192-0001LF
- added U1: ESP32-DEVKITC-32D, ESP32-DEVKITC-32D:MODULE_ESP32-DEVKITC-32D, symbol ESP32-DEVKITC-32D:ESP32-DEVKITC-32D
- added U2: MCP73831T-2ACI/OT, MCP73831T_2ACI_OT:SOT-23-5_MC_MCH, symbol MCP73831T_2ACI_OT:MCP73831T-2ACI_OT
- added U3: AP2112K-3.3TRG1, AP2112K_3_3TRG1:SOT95P285X140-5N, symbol AP2112K-3.3TRG1:AP2112K-3.3TRG1
- added U4: AD5941BCPZ-RL7, AD5941BCPZ_RL7:QFN50P700X700X80-49N, symbol AD5941BCPZ_RL7:AD5941BCPZ-RL7
- C10, C12, C8, C9: footprint HELPStat_V2:C0402 -> Capacitor_SMD:C_0402_1005Metric; Part Number (none) -> C0402C474K9PACTU
- C11: footprint HELPStat_V2:C0402 -> Capacitor_SMD:C_0402_1005Metric; Part Number (none) -> CL05A475KQ5NRNC
- C17, C3, C4, C5, C6: footprint HELPStat_V2:C0402 -> Capacitor_SMD:C_0402_1005Metric; Part Number (none) -> 0402W106M6R3HI
- C18, C19: footprint HELPStat_V2:C0402 -> Capacitor_SMD:C_0402_1005Metric; Part Number (none) -> CL05B104KP5NNNC
- C7: footprint HELPStat_V2:C0402 -> Capacitor_SMD:C_0402_1005Metric; Part Number (none) -> JMK105BJ105KV-F
- R4: footprint HELPStat_V2:R0603 -> Resistor_SMD:R_0603_1608Metric; Part Number (none) -> RR0816P-104-D
- R7, R8, R9: value 47k -> 4k7; footprint HELPStat_V2:R0402 -> Resistor_SMD:R_0402_1005Metric; Part Number (none) -> RC0402JR-074K7L
Connections:
- net CD2 is gone; now on net GND: R7.2
- net 3.3V: now also C20.1, C21.1, C22.1, U1.J2-1 (3V3), U3.5 (VOUT), U4.26 (IOVDD), U4.30 (AVDD), U4.6 (DVDD); no longer C17.1, C19.1, R7.1, R8.1
- net AFE.RST: now also U1.J2-10 (IO26), U4.22 (~{RESET})
- net AFE1: now also U4.34 (AFE1)
- net AFE2: now also U4.35 (AFE2)
- net AFE3: now also U4.27 (AFE3)
- net AFE4: now also U4.28 (AFE4)
- net AIN0: now also U4.39 (AIN0)
- net AIN1: now also U4.38 (AIN1)
- net AIN2: now also U4.37 (AIN2)
- net AIN3: now also U4.36 (AIN3/BUF_VREF1V8)
- net AIN4: now also U4.40 (AIN4/LPF0)
- net AVDD.REG: now also U4.5 (AVDD_REG)
- net BIAS.0: now also C19.1, U4.8 (VBIAS0)
- net BIAS.CAP: now also U4.31 (VBIAS_CAP)
- net BOOT: now also U1.J3-14 (IO0)
- net CE: now also U4.47 (CE0)
- net CS.AFE: now also U1.J2-11 (IO27), U4.15 (~{CS})
- net CS.SD: now also U1.J3-8 (IO19)
- net CS.SPI: now also U1.J3-6 (IO21)
- net DE: now also U4.46 (DE0)
- net DVDD.1V8: now also U4.14 (DVDD_REG_1V8)
- net GND: now also C20.2, C21.2, C22.2, J1.5 (GND), U1.J2-14 (GND1), U1.J3-1 (GND3), U1.J3-7 (GND2), U2.2 (VSS), U3.2 (GND), U4.13 (DGND), U4.23 (DGND__1), U4.25 (DGND__2), U4.29 (AGND), U4.42 (AGND__1), U4.44 (AGND_REF), U4.49 (EXP)
- net GPIO.0: now also U1.J2-9 (IO25), U4.19 (GPIO0)
- net GPIO.1: now also U4.20 (GPIO1)
- net GPIO.2: now also U4.21 (GPIO2)
- net MCU.RST: now also U1.J2-2 (EN)
- net MISO: now also U1.J3-12 (IO16), U4.18 (MISO); no longer R8.2
- net MOSI: now also U1.J3-9 (IO18), U4.17 (MOSI); no longer R9.2
- net RC0.0: now also U4.3 (RC0_0)
- net RC0.1: now also U4.2 (RC0_1)
- net RC0.2: now also U4.1 (RC0_2)
- net RCAL0: now also U4.32 (RCAL0)
- net RCAL1: now also U4.33 (RCAL1)
- net RE: now also U4.48 (RE0)
- net REF.1V8: now also U4.43 (VREF_1V8)
- net REF.2V5: now also U4.4 (VREF_2V5)
- net RX: now also U1.J3-5 (RXD0)
- net SCL/7/CH1: now also U1.J2-15 (IO13)
- net SCLK: now also U1.J3-11 (IO17), U4.16 (SCLK)
- net SDA/6/CH0: now also U1.J2-13 (IO12)
- net TX: now also U1.J3-4 (TXD0)
- net USB_N: now also J1.2 (D-), U1.J3-2 (IO23)
- net USB_P: now also J1.3 (D+), U1.J3-3 (IO22)
- net VLIPO: now also C17.1, U2.3 (VBAT)
- net VUSB: now also R8.1, D1.A, J1.1 (VUSB), U2.4 (VDD)
- net WE: now also U4.45 (SE0)
- net XTAL.I: now also U4.11 (XTALI)
- net XTAL.O: now also U4.12 (XTALO)
- net ZERO.0: now also U4.9 (VZERO0)
- net at C3.1, Q1.2 (S), TP3.P$1 (1): now also D1.C, U3.1 (VIN), U3.3 (EN)
- net at PWR0.A: now also R9.2
- new net: R7.1, U2.5 (PROG)
- new net: CHRG1.A, R8.2
- new net: CHRG1.C, U2.1 (STAT)
- no-connect marks 0 -> 19
Other:
- note added: "ESP32-DEVKITC-32D"
- note removed: "ESP32 S3 SWITCHES"

Commit message: Sch Draft Completed
Parts:
- removed CHRG1: YLW, HELPStat_V2:LED-0603, symbol HELPStat_V2-eagle-import:LED0603
- removed CS0: TPTP20SQ, HELPStat_V2:TP20SQ, symbol HELPStat_V2-eagle-import:TPTP20SQ
- removed ELECTRODES0, I2C0, SPI0, UART0: CONN_04, HELPStat_V2:1X04, symbol HELPStat_V2-eagle-import:CONN_04
- removed GPIOS/RST0, PERIPHERALS0: CONN_041.27MM, HELPStat_V2:1X04_1.27MM, symbol HELPStat_V2-eagle-import:CONN_041.27MM
- removed LIPO1: JST_2MM_MALE, HELPStat_V2:JST-2-SMD, symbol HELPStat_V2-eagle-import:JST_2MM_MALE
- removed PWR0: GREEN, HELPStat_V2:LED-0603, symbol HELPStat_V2-eagle-import:LED0603
- removed Q1: 2.5A/30V/105mΩ, HELPStat_V2:SOT23-3, symbol HELPStat_V2-eagle-import:PFET-DMG2307L
- removed RC0, XTAL0: CONN_02.50MIL, HELPStat_V2:1X02_1.27MM, symbol HELPStat_V2-eagle-import:CONN_02.50MIL
- removed RCAL0: CONN_02, HELPStat_V2:1X02, symbol HELPStat_V2-eagle-import:CONN_02
- removed TP3, TP4, UNK2V5, VB0, VCAP0, VZ0: TEST-POINT3X5, HELPStat_V2:PAD.03X.05, symbol HELPStat_V2-eagle-import:TEST-POINT3X5
- added CS0: TestPoint_Alt, TestPoint:TestPoint_Pad_2.0x2.0mm, symbol Connector:TestPoint_Alt
- added I2C0, J6, J7, J8, SPI0, UART0: M50-3530442, M50_3530442:HARWIN_M50-3530442, symbol M50-3530442:M50-3530442
- added J2: LIPO1, B2B_XH_A:JST_B2B-XH-A, symbol B2B-XH-A:B2B-XH-A
- added J3, J4, J5: M20-9990246, M20_9990246:HARWIN_M20-9990246, symbol M20-9990246:M20-9990246
- added LED1: YLW, LED_00-R18_OSR, symbol LED1212:GY_PSLM31.13-HQHS-5F5G-L2M2-100-R18
- added LED2: GRN, LED_00-R18_OSR, symbol LED1212:GY_PSLM31.13-HQHS-5F5G-L2M2-100-R18
- added MOSFET1: BSS205NH6327XTSA1, PG-SOT23-3-5_INF, symbol BSS205NH6327XTSA1:BSS205NH6327XTSA1
- added TP1, TP2, TP3, TP4, TP5, TP6: TestPoint, TestPoint:TestPoint_Pad_D1.0mm, symbol Connector:TestPoint
- H2, H4: value MOUNT-HOLE2.8 -> MOUNT-HOLE2.2; footprint HELPStat_V2:2,8 -> MountingHole:MountingHole_2.2mm_M2_Pad
Connections:
- net 3.3V: now also I2C0.1, TP2.1, UART0.1
- net AFE.RST: now also J6.4
- net AFE1: now also J7.4
- net AFE2: now also J7.3
- net AIN3: now also J7.2
- net AIN4: now also J7.1
- net BIAS.0: now also TP3.1
- net BIAS.CAP: now also TP5.1
- net CE: now also J8.2
- net CS.AFE: now also CS0.1
- net CS.SPI: now also SPI0.1
- net DE: now also J8.3
- net GND: now also I2C0.4, J2.1, LED2.1, UART0.4
- net GPIO.0: now also J6.1
- net GPIO.1: now also J6.2
- net GPIO.2: now also J6.3
- net MISO: now also SPI0.2
- net MOSI: now also SPI0.4
- net RC0.0: now also J5.1
- net RC0.1: now also J5.2
- net RCAL0: now also J3.1
- net RCAL1: now also J3.2
- net RE: now also J8.1
- net REF.2V5: now also TP6.1
- net RX: now also UART0.2
- net SCL/7/CH1: now also I2C0.3
- net SCLK: now also SPI0.3
- net SDA/6/CH0: now also I2C0.2
- net TX: now also UART0.3
- net VLIPO: now also J2.2, MOSFET1.3 (D)
- net VUSB: now also MOSFET1.1 (G)
- net WE: now also J8.4
- net XTAL.I: now also J4.1
- net XTAL.O: now also J4.2
- net ZERO.0: now also TP4.1
- net at R8.2: now also LED1.2
- net at U2.1 (STAT): now also LED1.1
- net at C3.1, D1.C, U3.1 (VIN)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: now also MOSFET1.2 (S), TP1.1
- net at R9.2: now also LED2.2

Commit message: CSV and SCH edits
Parts:
- C17, C3, C4, C5, C6: Part Number 0402W106M6R3HI -> CL05A106MP5NUNC
Changed lines of the file:
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@@
 			)
 		)
-		(property "Part Number" "0402W106M6R3HI"
+		(property "Part Number" "CL05A106MP5NUNC"
 			(at 177.8 160.02 0)
 			(effects
@@
 			)
 		)
-		(property "Part Number" "0402W106M6R3HI"
+		(property "Part Number" "CL05A106MP5NUNC"
 			(at 119.38 195.58 0)
 			(effects
@@
 			)
 		)
-		(property "Part Number" "0402W106M6R3HI"
+		(property "Part Number" "CL05A106MP5NUNC"
 			(at 123.19 129.54 0)
 			(effects
@@
 			)
 		)
-		(property "Part Number" "0402W106M6R3HI"
+		(property "Part Number" "CL05A106MP5NUNC"
 			(at 68.58 198.12 0)
 			(effects
@@
 			)
 		)
-		(property "Part Number" "0402W106M6R3HI"
+		(property "Part Number" "CL05A106MP5NUNC"
 			(at 190.5 160.02 0)
 			(effects

Commit message: pcb v2
Parts:
- removed U1: ESP32-DEVKITC-32D, ESP32-DEVKITC-32D:MODULE_ESP32-DEVKITC-32D, symbol ESP32-DEVKITC-32D:ESP32-DEVKITC-32D
- added H1, H3: MOUNT-HOLE2.2, MountingHole:MountingHole_2.2mm_M2_Pad, symbol HELPStat_V2-eagle-import:MOUNT-HOLE2.8
- added U5: ESP32-S3-DEVKITC-1-N8R2, ESP32-S3-DEVKITC-1-N8R2:XCVR_ESP32-S3-DEVKITC-1-N8R2, symbol ESP32-S3-DEVKITC-1-N8R2:ESP32-S3-DEVKITC-1-N8R2
- C10, C12, C8, C9: footprint Capacitor_SMD:C_0402_1005Metric -> Capacitor_SMD:C_0603_1608Metric; Part Number C0402C474K9PACTU -> TMK107B7474KA-TR
- C11: footprint Capacitor_SMD:C_0402_1005Metric -> Capacitor_SMD:C_0603_1608Metric; Part Number CL05A475KQ5NRNC -> LMK107BJ475KA-T
- C17, C3, C4, C5, C6: footprint Capacitor_SMD:C_0402_1005Metric -> Capacitor_SMD:C_0603_1608Metric; Part Number CL05A106MP5NUNC -> LMK107BBJ106MALT
- C18, C19, C20, C21, C22: footprint Capacitor_SMD:C_0402_1005Metric -> Capacitor_SMD:C_0603_1608Metric; Part Number CL05B104KP5NNNC -> CC0603KRX7R7BB104
- C7: footprint Capacitor_SMD:C_0402_1005Metric -> Capacitor_SMD:C_0603_1608Metric; Part Number JMK105BJ105KV-F -> CL10B105KP8NNNC
- R4: Part Number RR0816P-104-D -> RC0603FR-07100KL
- R7, R8, R9: footprint Resistor_SMD:R_0402_1005Metric -> Resistor_SMD:R_0603_1608Metric; Part Number RC0402JR-074K7L -> RC0603FR-074K7L
Connections:
- net 3.3V: now also U5.J1_1 (3V3), U5.J1_2 (3V3)
- net AFE.RST: now also U5.J1_16 (GPIO10)
- net BOOT: now also U5.J3_14 (GPIO0)
- net CS.AFE: now also U5.J1_17 (GPIO11)
- net CS.SD: now also U5.J3_18 (GPIO21)
- net CS.SPI: now also U5.J3_10 (GPIO38)
- net GND: now also U5.J1_22 (GND), U5.J3_1 (GND), U5.J3_21 (GND), U5.J3_22 (GND)
- net GPIO.0: now also U5.J1_15 (GPIO9)
- net MCU.RST: now also U5.J1_3 (RST)
- net MISO: now also U5.J3_11 (GPIO37)
- net MOSI: now also U5.J3_13 (GPIO35)
- net RX: now also U5.J3_3 (U0RXD/GPIO44)
- net SCLK: now also U5.J3_12 (GPIO36)
- net TX: now also U5.J3_2 (U0TXD/GPIO43)
- net USB_N: now also U5.J3_20 (USB_D-/GPIO19)
- net USB_P: now also U5.J3_19 (USB_D+/GPIO20)
- new net SCL/7/CH1: U5.J1_7 (GPIO7)
- new net SDA/6/CH0: U5.J1_6 (GPIO6)
- no-connect marks 19 -> 1
Other:
- moved on the sheet: C5, C7

Commit message: Sch and PCB cleanup/fixes
Parts:
- I2C0, J6, J7, J8, SPI0, UART0: value M50-3530442 -> 61300411121; footprint M50_3530442:HARWIN_M50-3530442 -> 61300411121:61300411121; MANUFACTURER HARWIN -> (none); Part Number M50-3530442 -> 61300411121
- U5: Part Number (none) -> ESP32-S3-DEVKITC-1-N8R2
Changed lines of the file:
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@@
 			)
 		)
+		(property "Part Number" "ESP32-S3-DEVKITC-1-N8R2"
+			(at 209.55 180.34 0)
+			(effects
+				(font
+					(size 1.27 1.27)
+				)
+				(hide yes)
+			)
+		)
 		(property "MF" "Espressif Systems"
 			(at 209.55 180.34 0)
@@
 			)
 		)
-		(property "Value" "M50-3530442"
+		(property "Value" "61300411121"
 			(at 267.97 96.5199 0)
 			(effects
@@
 			)
 		)
-		(property "Footprint" "M50_3530442:HARWIN_M50-3530442"
+		(property "Footprint" "61300411121:61300411121"
 			(at 260.35 96.52 0)
 			(effects
@@
 			)
 		)
-		(property "Part Number" "M50-3530442"
+		(property "Part Number" "61300411121"
 			(at 260.35 96.52 0)
 			(effects
@@
 			)
 		)
-		(property "MANUFACTURER" "HARWIN"
+		(property "MANUFACTURER" ""
 			(at 260.35 96.52 0)
 			(effects
@@
 			)
 		)
-		(property "Value" "M50-3530442"
+		(property "Value" "61300411121"
 			(at 438.15 198.1199 0)
 			(effects
@@
 			)
 		)
-		(property "Footprint" "M50_3530442:HARWIN_M50-3530442"
+		(property "Footprint" "61300411121:61300411121"
 			(at 430.53 198.12 0)
 			(effects
@@
 			)
 		)
-		(property "Part Number" "M50-3530442"
+		(property "Part Number" "61300411121"
 			(at 430.53 198.12 0)
 			(effects
@@
 			)
 		)
-		(property "MANUFACTURER" "HARWIN"
+		(property "MANUFACTURER" ""
 			(at 430.53 198.12 0)
 			(effects
@@
 			)
 		)
-		(property "Value" "M50-3530442"
+		(property "Value" "61300411121"
 			(at 229.87 96.5199 0)
 			(effects
@@
 			)
 		)
-		(property "Footprint" "M50_3530442:HARWIN_M50-3530442"
+		(property "Footprint" "61300411121:61300411121"
 			(at 222.25 96.52 0)
 			(effects
@@
 			)
 		)
-		(property "Part Number" "M50-3530442"
+		(property "Part Number" "61300411121"
 			(at 222.25 96.52 0)
 			(effects
@@
 			)
 		)
-		(property "MANUFACTURER" "HARWIN"
+		(property "MANUFACTURER" ""
 			(at 222.25 96.52 0)
 			(effects
@@
 			)
 		)
-		(property "Value" "M50-3530442"
+		(property "Value" "61300411121"
 			(at 438.15 177.7999 0)
 			(effects
@@
 			)
 		)
-		(property "Footprint" "M50_3530442:HARWIN_M50-3530442"
+		(property "Footprint" "61300411121:61300411121"
 			(at 430.53 177.8 0)
 			(effects
@@
 			)
 		)
-		(property "Part Number" "M50-3530442"
+		(property "Part Number" "61300411121"
 			(at 430.53 177.8 0)
 			(effects
@@
 			)
 		)
-		(property "MANUFACTURER" "HARWIN"
+		(property "MANUFACTURER" ""
 			(at 430.53 177.8 0)
 			(effects
@@
 			)
 		)
-		(property "Value" "M50-3530442"
+		(property "Value" "61300411121"
 			(at 229.87 119.3799 0)
 			(effects
@@
 			)
 		)
-		(property "Footprint" "M50_3530442:HARWIN_M50-3530442"
+		(property "Footprint" "61300411121:61300411121"
 			(at 222.25 119.38 0)
 			(effects
@@
 			)
 		)
-		(property "Part Number" "M50-3530442"
+		(property "Part Number" "61300411121"
 			(at 222.25 119.38 0)
 			(effects
@@
 			)
 		)
-		(property "MANUFACTURER" "HARWIN"
+		(property "MANUFACTURER" ""
 			(at 222.25 119.38 0)
 			(effects
@@
 			)
 		)
-		(property "Value" "M50-3530442"
+		(property "Value" "61300411121"
 			(at 472.44 198.1199 0)
 			(effects
@@
 			)
 		)
-		(property "Footprint" "M50_3530442:HARWIN_M50-3530442"
+		(property "Footprint" "61300411121:61300411121"
 			(at 464.82 198.12 0)
 			(effects
@@
 			)
 		)
-		(property "Part Number" "M50-3530442"
+		(property "Part Number" "61300411121"
 			(at 464.82 198.12 0)
 			(effects
@@
 			)
 		)
-		(property "MANUFACTURER" "HARWIN"
+		(property "MANUFACTURER" ""
 			(at 464.82 198.12 0)
 			(effects
