File: Helpstat/HELPStat_V2.kicad_pcb (KiCad board)
At the start: 2 copper layers, 102 x 45 mm, 51 parts, among them J1 10118192-0001LF, J2 LIPO1, J3 M20-9990246, J4 M20-9990246, J5 M20-9990246, J6 M50-3530442, J7 M50-3530442, J8 M50-3530442, U2 MCP73831T-2ACI/OT, U3 AP2112K-3.3TRG1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

Commit message: Sch and PCB cleanup/fixes
Parts:
- removed _: LOGO, Dome:Dome of Protection
- added G***: LOGO, ConduitQ:Radiant Transfer, F.Cu at (127.8, 118.5)
- I2C0, J6, J7, J8, SPI0, UART0: value M50-3530442 -> 61300411121; footprint M50_3530442:HARWIN_M50-3530442 -> 61300411121:61300411121
- moved I2C0 14.8 mm to (68.5, 94.5)
- moved C3 3.59 mm to (100.5, 119.5)
- moved J7 3.05 mm to (120.2, 116.0)
- moved J8 2.92 mm to (124.0, 102.2)
- moved SPI0 1.11 mm to (63.7, 128.2)
- moved UART0 0.83 mm to (86.5, 128.2)
- moved H2 0.50 mm to (134.0, 93.0)
- moved H3 0.50 mm to (39.0, 131.0)
Routing:
- net /SDA/6/CH0: track 25.6 -> 10.0 mm
- net /SCL/7/CH1: track 24.2 -> 10.0 mm
- net 3.3V: track 124.3 -> 114.3 mm
- net /AFE1: track 8.26 -> 12.0 mm
- net /AFE.RST: track 67.4 -> 70.8 mm
- net /AFE2: track 7.15 -> 10.2 mm
- net /AIN3: track 5.88 -> 8.40 mm
- net /AIN4: track 5.57 -> 7.57 mm
- net /RE: track 11.6 -> 13.3 mm
- net /CE: track 11.3 -> 12.5 mm
- net /GPIO.1: track 6.39 -> 5.27 mm
- net Net-(MOSFET1-S): track 17.4 -> 16.4 mm
- net /GPIO.0: track 60.3 -> 59.6 mm
- net /DE: track 11.0 -> 11.7 mm
- net /SCLK: track 56.2 -> 56.9 mm
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
Commit message: extra PCB changes
Parts:
- moved G*** 5.84 mm to (133.5, 119.5)
- moved H2 1.58 mm to (132.5, 92.5)
- moved H1 1.12 mm to (40.0, 92.5)
- moved R7 0.50 mm to (124.5, 125.5)
Routing:
- net GND: track 65.6 -> 70.0 mm, vias 15 -> 19
Other:
- board text added: "CE"
- board text added: "DE"
- board text added: "RE"
- board text added: "WE"
